Commit message: BEV planning

File: src/sim/robot_description/urdf/turtlebot3_burger.urdf.xacro (robot description, xacro)
@@ -3,4 +3,5 @@
   <!-- Arguments -->
   <xacro:arg name="namespace" default=""/>
+  <xacro:arg name="use_lidar" default="true"/>
   <xacro:property name="ns" value="$(arg namespace)"/>
   <!-- ===================== -->
@@ -23,5 +24,5 @@
       <origin xyz="-0.032 0 0"/>
       <geometry>
-        <mesh filename="package://robot_description/meshes/turtlebot3_description/meshes/bases/burger_base.stl"
+        <mesh filename="package://sim/robot_description/meshes/turtlebot3_description/meshes/bases/burger_base.stl"
               scale="0.001 0.001 0.001"/>
       </geometry>
@@ -56,5 +57,5 @@
       <origin rpy="1.57 0 0"/>
       <geometry>
-        <mesh filename="package://robot_description/meshes/turtlebot3_description/meshes/wheels/left_tire.stl"
+        <mesh filename="package://sim/robot_description/meshes/turtlebot3_description/meshes/wheels/left_tire.stl"
               scale="0.001 0.001 0.001"/>
       </geometry>
@@ -85,5 +86,5 @@
       <origin rpy="1.57 0 0"/>
       <geometry>
-        <mesh filename="package://robot_description/meshes/turtlebot3_description/meshes/wheels/right_tire.stl"
+        <mesh filename="package://sim/robot_description/meshes/turtlebot3_description/meshes/wheels/right_tire.stl"
               scale="0.001 0.001 0.001"/>
       </geometry>
@@ -124,5 +125,5 @@
     <visual>
       <geometry>
-        <mesh filename="package://robot_description/meshes/turtlebot3_description/meshes/sensors/lds.stl"
+        <mesh filename="package://sim/robot_description/meshes/turtlebot3_description/meshes/sensors/lds.stl"
               scale="0.001 0.001 0.001"/>
       </geometry>
@@ -145,27 +146,29 @@
     <!-- ============================================================= -->
     <!-- Gazebo Sensor Plugins -->
-    <gazebo reference="${ns}base_scan">
-      <sensor name="lidar" type="gpu_lidar">
-        <pose>0 0 0 0 0 0</pose>
-        <topic>scan</topic>
-        <update_rate>5</update_rate>
-        <ray>
-          <scan>
-            <horizontal>
-              <samples>360</samples>
-              <resolution>1</resolution>
-              <min_angle>0.0</min_angle>
-              <max_angle>6.28318</max_angle>
-            </horizontal>
-          </scan>
-          <range>
-            <min>0.12</min>
-            <max>3.5</max>
-          </range>
-        </ray>
-        <always_on>true</always_on>
-        <visualize>true</visualize>
-      </sensor>
-    </gazebo>
+    <xacro:if value="$(arg use_lidar)">
+      <gazebo reference="${ns}base_scan">
+        <sensor name="lidar" type="gpu_lidar">
+          <pose>0 0 0 0 0 0</pose>
+          <topic>scan</topic>
+          <update_rate>5</update_rate>
+          <ray>
+            <scan>
+              <horizontal>
+                <samples>360</samples>
+                <resolution>1</resolution>
+                <min_angle>0.0</min_angle>
+                <max_angle>6.28318</max_angle>
+              </horizontal>
+            </scan>
+            <range>
+              <min>0.12</min>
+              <max>3.5</max>
+            </range>
+          </ray>
+          <always_on>true</always_on>
+          <visualize>true</visualize>
+        </sensor>
+      </gazebo>
+    </xacro:if>
     <!-- ================= Gazebo Harmonic DiffDrive ================= -->
     <gazebo>
@@ -180,6 +183,6 @@
         <wheel_radius>0.033</wheel_radius>
         <!-- ROS interface -->
-        <topic>cmd_vel</topic>
-        <odom_topic>odom</odom_topic>
+        <topic>/model/turtlebot3/cmd_vel</topic>
+        <odom_topic>/model/turtlebot3/odometry</odom_topic>
         <!-- Frames -->
         <frame_id>odom</frame_id>

Commit message: New attempts for paper, still messy

File: src/sim/robot_description/urdf/turtlebot3_burger.urdf.xacro (robot description, xacro)
@@ -142,4 +142,37 @@
         iyy="0.001" iyz="0.0"
         izz="0.001"/>
+    </inertial>
+  </link>
+  <!-- ===================== -->
+  <!-- Fiducial Marker       -->
+  <!-- ===================== -->
+  <!--
+    Top-mounted ArUco marker for external camera detection.
+    The plane faces +Z so overhead/oblique external cameras can detect it.
+  -->
+  <joint name="${ns}aruco_marker_joint" type="fixed">
+    <parent link="${ns}base_link"/>
+    <child link="${ns}aruco_marker_link"/>
+    <origin xyz="0.020 0.000 0.215" rpy="0 0 0"/>
+  </joint>
+  <link name="${ns}aruco_marker_link">
+    <visual>
+      <geometry>
+        <mesh filename="package://sim/robot_description/meshes/aruco/aruco_4x4_50_id0.dae"
+              scale="0.50 0.50 1.0"/>
+      </geometry>
+    </visual>
+    <collision>
+      <geometry>
+        <box size="0.50 0.50 0.001"/>
+      </geometry>
+    </collision>
+    <inertial>
+      <mass value="0.001"/>
+      <origin xyz="0 0 0"/>
+      <inertia
+        ixx="1e-7" ixy="0.0" ixz="0.0"
+        iyy="1e-7" iyz="0.0"
+        izz="1e-7"/>
     </inertial>
   </link>

Commit message: Occlusion objects added

File: src/sim/robot_description/urdf/turtlebot3_burger.urdf.xacro (robot description, xacro)
@@ -11,4 +11,6 @@
   <material name="dark"><color rgba="0.3 0.3 0.3 1"/></material>
   <material name="light_black"><color rgba="0.4 0.4 0.4 1"/></material>
+  <material name="front_red"><color rgba="0.98 0.08 0.08 1.0"/></material>
+  <material name="rear_blue"><color rgba="0.05 0.20 0.98 1.0"/></material>
   <!-- ===================== -->
   <!-- Base -->
@@ -29,4 +31,19 @@
       <material name="light_black"/>
     </visual>
+    <!-- High-contrast orientation panels for external camera tracking -->
+    <visual>
+      <origin xyz="0.075 0.000 0.162"/>
+      <geometry>
+        <box size="0.120 0.110 0.018"/>
+      </geometry>
+      <material name="front_red"/>
+    </visual>
+    <visual>
+      <origin xyz="-0.085 0.000 0.162"/>
+      <geometry>
+        <box size="0.100 0.110 0.018"/>
+      </geometry>
+      <material name="rear_blue"/>
+    </visual>
     <collision>
       <origin xyz="-0.032 0 0.070"/>
@@ -142,37 +159,4 @@
         iyy="0.001" iyz="0.0"
         izz="0.001"/>
-    </inertial>
-  </link>
-  <!-- ===================== -->
-  <!-- Fiducial Marker       -->
-  <!-- ===================== -->
-  <!--
-    Top-mounted ArUco marker for external camera detection.
-    The plane faces +Z so overhead/oblique external cameras can detect it.
-  -->
-  <joint name="${ns}aruco_marker_joint" type="fixed">
-    <parent link="${ns}base_link"/>
-    <child link="${ns}aruco_marker_link"/>
-    <origin xyz="0.020 0.000 0.215" rpy="0 0 0"/>
-  </joint>
-  <link name="${ns}aruco_marker_link">
-    <visual>
-      <geometry>
-        <mesh filename="package://sim/robot_description/meshes/aruco/aruco_4x4_50_id0.dae"
-              scale="0.50 0.50 1.0"/>
-      </geometry>
-    </visual>
-    <collision>
-      <geometry>
-        <box size="0.50 0.50 0.001"/>
-      </geometry>
-    </collision>
-    <inertial>
-      <mass value="0.001"/>
-      <origin xyz="0 0 0"/>
-      <inertia
-        ixx="1e-7" ixy="0.0" ixz="0.0"
-        iyy="1e-7" iyz="0.0"
-        izz="1e-7"/>
     </inertial>
   </link>

Commit message: Robout colour detection

File: src/sim/robot_description/urdf/turtlebot3_burger.urdf.xacro (robot description, xacro)
@@ -29,20 +29,5 @@
               scale="0.001 0.001 0.001"/>
       </geometry>
-      <material name="light_black"/>
-    </visual>
-    <!-- High-contrast orientation panels for external camera tracking -->
-    <visual>
-      <origin xyz="0.075 0.000 0.162"/>
-      <geometry>
-        <box size="0.120 0.110 0.018"/>
-      </geometry>
       <material name="front_red"/>
-    </visual>
-    <visual>
-      <origin xyz="-0.085 0.000 0.162"/>
-      <geometry>
-        <box size="0.100 0.110 0.018"/>
-      </geometry>
-      <material name="rear_blue"/>
     </visual>
     <collision>
@@ -141,9 +126,10 @@
   <link name="${ns}base_scan">
     <visual>
+      <origin xyz="-0.045 0 0"/>
       <geometry>
         <mesh filename="package://sim/robot_description/meshes/turtlebot3_description/meshes/sensors/lds.stl"
               scale="0.001 0.001 0.001"/>
       </geometry>
-      <material name="dark"/>
+      <material name="rear_blue"/>
     </visual>
     <collision>

Commit message: Ugly push

File: src/sim/robot_description/urdf/turtlebot3_burger.urdf.xacro (robot description, xacro)
@@ -5,4 +5,17 @@
   <xacro:arg name="use_lidar" default="true"/>
   <xacro:property name="ns" value="$(arg namespace)"/>
+  <!-- Pose-keypoint definitions (in base_link frame). No extra geometry is
+       added: the keypoints are virtual points anchored on the existing
+       robot. The blue lidar (rear_blue material on the lds.stl mesh) is the
+       visible "rear" feature; the red base mesh (front_red on burger_base.stl)
+       extends forward of the lidar, providing the heading cue. The model
+       learns to predict both keypoints at the same world Z so the state node
+       can back-project them to a single z-plane without bias.
+       World Z given a base_footprint at z=robot_z is:
+         z_world = robot_z + base_joint_z(0.010) + pm_marker_z. -->
+  <xacro:property name="pm_front_x" value="0.050"/>
+  <xacro:property name="pm_rear_x"  value="-0.032"/>
+  <xacro:property name="pm_marker_y" value="0.0"/>
+  <xacro:property name="pm_marker_z" value="0.188"/>
   <!-- ===================== -->
   <!-- Materials (REQUIRED) -->

Commit message: runtime changes

File: src/sim/robot_description/urdf/turtlebot3_burger.urdf.xacro (robot description, xacro)
@@ -14,8 +14,12 @@
        World Z given a base_footprint at z=robot_z is:
          z_world = robot_z + base_joint_z(0.010) + pm_marker_z. -->
-  <xacro:property name="pm_front_x" value="0.050"/>
-  <xacro:property name="pm_rear_x"  value="-0.032"/>
+  <!-- v2: explicit small marker disks at MAX front-rear separation (cyan front /
+       magenta rear), replacing the old virtual centroids of the big red base /
+       blue lidar. Baseline 0.140 m (was 0.082) + small precise distinct markers
+       => tighter heading, lower view-dependent bias, no front/rear flips. -->
+  <xacro:property name="pm_front_x" value="0.040"/>
+  <xacro:property name="pm_rear_x"  value="-0.100"/>
   <xacro:property name="pm_marker_y" value="0.0"/>
-  <xacro:property name="pm_marker_z" value="0.188"/>
+  <xacro:property name="pm_marker_z" value="0.200"/>
   <!-- ===================== -->
   <!-- Materials (REQUIRED) -->
@@ -26,4 +30,6 @@
   <material name="front_red"><color rgba="0.98 0.08 0.08 1.0"/></material>
   <material name="rear_blue"><color rgba="0.05 0.20 0.98 1.0"/></material>
+  <material name="marker_cyan"><color rgba="0.0 0.95 0.95 1.0"/></material>
+  <material name="marker_magenta"><color rgba="0.95 0.0 0.95 1.0"/></material>
   <!-- ===================== -->
   <!-- Base -->
@@ -158,4 +164,39 @@
         iyy="0.001" iyz="0.0"
         izz="0.001"/>
+    </inertial>
+  </link>
+  <!-- ===================== -->
+  <!-- Heading marker disks (v2): small distinct top markers at max front-rear
+       separation. front=cyan @ pm_front_x, rear=magenta @ pm_rear_x, both at
+       pm_marker_z (above the lidar so the oblique camera sees both). -->
+  <!-- ===================== -->
+  <joint name="${ns}front_marker_joint" type="fixed">
+    <parent link="${ns}base_link"/>
+    <child link="${ns}front_marker"/>
+    <origin xyz="${pm_front_x} ${pm_marker_y} ${pm_marker_z}"/>
+  </joint>
+  <link name="${ns}front_marker">
+    <visual>
+      <geometry><cylinder length="0.008" radius="0.025"/></geometry>
+      <material name="marker_cyan"/>
+    </visual>
+    <inertial>
+      <mass value="0.001"/>
+      <inertia ixx="1e-7" ixy="0" ixz="0" iyy="1e-7" iyz="0" izz="1e-7"/>
+    </inertial>
+  </link>
+  <joint name="${ns}rear_marker_joint" type="fixed">
+    <parent link="${ns}base_link"/>
+    <child link="${ns}rear_marker"/>
+    <origin xyz="${pm_rear_x} ${pm_marker_y} ${pm_marker_z}"/>
+  </joint>
+  <link name="${ns}rear_marker">
+    <visual>
+      <geometry><cylinder length="0.008" radius="0.025"/></geometry>
+      <material name="marker_magenta"/>
+    </visual>
+    <inertial>
+      <mass value="0.001"/>
+      <inertia ixx="1e-7" ixy="0" ixz="0" iyy="1e-7" iyz="0" izz="1e-7"/>
     </inertial>
   </link>

Commit message: New Q

File: src/sim/robot_description/urdf/turtlebot3_burger.urdf.xacro (robot description, xacro)
@@ -4,4 +4,5 @@
   <xacro:arg name="namespace" default=""/>
   <xacro:arg name="use_lidar" default="true"/>
+  <xacro:arg name="show_pose_markers" default="false"/>
   <xacro:property name="ns" value="$(arg namespace)"/>
   <!-- Pose-keypoint definitions (in base_link frame). No extra geometry is
@@ -169,36 +170,40 @@
   <!-- Heading marker disks (v2): small distinct top markers at max front-rear
        separation. front=cyan @ pm_front_x, rear=magenta @ pm_rear_x, both at
-       pm_marker_z (above the lidar so the oblique camera sees both). -->
-  <!-- ===================== -->
-  <joint name="${ns}front_marker_joint" type="fixed">
-    <parent link="${ns}base_link"/>
-    <child link="${ns}front_marker"/>
-    <origin xyz="${pm_front_x} ${pm_marker_y} ${pm_marker_z}"/>
-  </joint>
-  <link name="${ns}front_marker">
-    <visual>
-      <geometry><cylinder length="0.008" radius="0.025"/></geometry>
-      <material name="marker_cyan"/>
-    </visual>
-    <inertial>
-      <mass value="0.001"/>
-      <inertia ixx="1e-7" ixy="0" ixz="0" iyy="1e-7" iyz="0" izz="1e-7"/>
-    </inertial>
-  </link>
-  <joint name="${ns}rear_marker_joint" type="fixed">
-    <parent link="${ns}base_link"/>
-    <child link="${ns}rear_marker"/>
-    <origin xyz="${pm_rear_x} ${pm_marker_y} ${pm_marker_z}"/>
-  </joint>
-  <link name="${ns}rear_marker">
-    <visual>
-      <geometry><cylinder length="0.008" radius="0.025"/></geometry>
-      <material name="marker_magenta"/>
-    </visual>
-    <inertial>
-      <mass value="0.001"/>
-      <inertia ixx="1e-7" ixy="0" ixz="0" iyy="1e-7" iyz="0" izz="1e-7"/>
-    </inertial>
-  </link>
+       pm_marker_z (above the lidar so the oblique camera sees both).
+       They are opt-in so segmentation-detector runs keep the visual domain used
+       to train aws_yolo_simseg_v2. -->
+  <!-- ===================== -->
+  <xacro:if value="$(arg show_pose_markers)">
+    <joint name="${ns}front_marker_joint" type="fixed">
+      <parent link="${ns}base_link"/>
+      <child link="${ns}front_marker"/>
+      <origin xyz="${pm_front_x} ${pm_marker_y} ${pm_marker_z}"/>
+    </joint>
+    <link name="${ns}front_marker">
+      <visual>
+        <geometry><cylinder length="0.008" radius="0.025"/></geometry>
+        <material name="marker_cyan"/>
+      </visual>
+      <inertial>
+        <mass value="0.001"/>
+        <inertia ixx="1e-7" ixy="0" ixz="0" iyy="1e-7" iyz="0" izz="1e-7"/>
+      </inertial>
+    </link>
+    <joint name="${ns}rear_marker_joint" type="fixed">
+      <parent link="${ns}base_link"/>
+      <child link="${ns}rear_marker"/>
+      <origin xyz="${pm_rear_x} ${pm_marker_y} ${pm_marker_z}"/>
+    </joint>
+    <link name="${ns}rear_marker">
+      <visual>
+        <geometry><cylinder length="0.008" radius="0.025"/></geometry>
+        <material name="marker_magenta"/>
+      </visual>
+      <inertial>
+        <mass value="0.001"/>
+        <inertia ixx="1e-7" ixy="0" ixz="0" iyy="1e-7" iyz="0" izz="1e-7"/>
+      </inertial>
+    </link>
+  </xacro:if>
     <!-- ============================================================= -->
     <!-- Gazebo Sensor Plugins -->
