Commit message: Repair the EFE planner objective and lock its constants
The planner's no-go term reached 1e6 on routes the footprint validator called
clear, which made route cost a no-go ranking rather than an EFE ranking. Three
defects caused it, each fixed here by deriving the constant from a measured
quantity rather than choosing it:

- nogo_safe_distance 0.55 -> 0.325 (robot half-width 0.275 plus a 0.05
  lane-keeping margin). The old value was the circumscribed radius, which left
  the 1.10 m lanes a negative lateral budget, i.e. infeasible before any
  uncertainty existed.
- nogo_logbarrier_eps 1e-3 -> 0.05, equal to nogo_warning_band. At 1e-3 a 1 mm
  notional violation cost more than the entire risk term.
- use_belief_nogo_cost now defaults true. With it off the obstacle term saw only
  the mean path, so predicted belief growth cost nothing.

With the no-go term no longer masking it, the risk term was a squared distance
to the goal: network_goal_std_m 0.15 made the objective a shortest-path planner
with a small entropy correction. Set to 0.35, the declared goal_success_radius.

The ambiguity term now implements Kouw (IWAI 2024) Lemma 1 under the first-order
extended transform of Theorem 1, evaluated on an availability-weighted
commissioned covariance. Theorem 1 makes this constant over states for a fixed
sensor; it varies here only because commissioning makes R and q spatial fields.
Hand, NumPy and CasADi paths agree to 1e-6 per pose and 1e-3 over a rollout.

Two accounting bugs are fixed. The objective summed a fixed horizon regardless
of route duration, so a short route banked its remaining steps parked at the
goal and accumulated that cell's ambiguity; a smooth arrival gate now zeroes
every term after arrival. Summed per-step terms also silently encode route
length, so per-step values must be inspected along a route, never only totals.

Process noise is set to conservatively bound the simulated odometry drift, and
the encoder noise is raised to a low-traction warehouse condition: the previous
setting produced 1.3-2.2% position drift per metre, inside the 0.50-2.30% band
published for calibrated wheel odometry on good surfaces. UnicyclePlannerBase
now warns if either process-noise value is overridden.

docs/PLANNER_LOCK.md and docs/PROCESS_NOISE_LOCK.md record every value with its
derivation. Stale planning and status documents are removed; they described
superseded method decisions and were being read as current.

Route choice is currently a null: on 11 of 11 contrast tasks both arms select
the same route. Earlier positive results predate the arrival-gate fix and are
retracted.

Co-Authored-By: Claude Opus 5 (1M context) <noreply@anthropic.com>

File: src/sim/robot_description/urdf/warehouse_amr.urdf.xacro (robot description, xacro)
@@ -6,5 +6,5 @@
          body      0.800 x 0.550 m, deck top at 0.350 m
          wheels    r 0.100, separation 0.440, differential, casters fore/aft
-         livery    charcoal chassis, hazard-yellow bumper band, grey load deck
+         livery    saturated blue chassis/deck, hazard-yellow bumper band
        No saturated marker disks: heading is carried by the chassis itself.
        Seen from an oblique ceiling camera the front has a recessed sensor
@@ -40,9 +40,13 @@
   <!-- Materials -->
   <!-- ===================== -->
-  <material name="chassis_charcoal"><color rgba="0.16 0.17 0.19 1.0"/></material>
-  <material name="deck_grey"><color rgba="0.55 0.56 0.58 1.0"/></material>
+  <!-- The detector target is deliberately blue, but it keeps three blue tones,
+       the yellow bumper and black sensor features so heading/shape remain
+       visible. Blue drums and totes in the warehouse are retained as hard
+       negatives; colour alone must never be sufficient for detection. -->
+  <material name="chassis_blue"><color rgba="0.04 0.20 0.62 1.0"/></material>
+  <material name="deck_blue"><color rgba="0.08 0.42 0.90 1.0"/></material>
   <material name="hazard_yellow"><color rgba="0.85 0.65 0.05 1.0"/></material>
   <material name="sensor_black"><color rgba="0.06 0.06 0.07 1.0"/></material>
-  <material name="cabinet_grey"><color rgba="0.33 0.34 0.36 1.0"/></material>
+  <material name="cabinet_blue"><color rgba="0.03 0.30 0.76 1.0"/></material>
   <material name="dark"><color rgba="0.3 0.3 0.3 1"/></material>
   <!-- ===================== -->
@@ -64,5 +68,5 @@
       <origin xyz="0 0 0.195"/>
       <geometry><box size="${body_l} ${body_w} 0.230"/></geometry>
-      <material name="chassis_charcoal"/>
+      <material name="chassis_blue"/>
     </visual>
     <collision>
@@ -105,5 +109,5 @@
   <xacro:trim name="deck" xyz="0 0 0.325"
               size="${body_l - 0.020} ${body_w - 0.020} 0.030"
-              material="deck_grey"/>
+              material="deck_blue"/>
   <!-- FRONT cue: recessed sensor bar across the leading face -->
   <xacro:trim name="sensor_bar" xyz="0.392 0 0.250"
@@ -116,5 +120,5 @@
   <!-- REAR cue: raised control cabinet, the tallest thing on the deck -->
   <xacro:trim name="cabinet" xyz="-0.280 0 0.365"
-              size="0.170 0.300 0.050" material="cabinet_grey"/>
+              size="0.170 0.300 0.050" material="cabinet_blue"/>
   <!-- ===================== -->
   <!-- Drive wheels -->
@@ -163,5 +167,4 @@
       <collision>
         <geometry><sphere radius="0.040"/></geometry>
-        <surface><friction><ode><mu>0.05</mu><mu2>0.05</mu2></ode></friction></surface>
       </collision>
       <inertial>
@@ -170,4 +173,10 @@
       </inertial>
     </link>
+    <!-- URDF collision <surface> is discarded by sdformat. Gazebo reference
+         extensions preserve the intended low caster friction after lumping. -->
+    <gazebo reference="${ns}${name}_link">
+      <mu1>0.05</mu1>
+      <mu2>0.05</mu2>
+    </gazebo>
   </xacro:macro>
   <xacro:caster name="caster_front" x="0.300"/>

Commit message: Remove contact sensing from the world, robot and launch; one world
Collisions are scored offline as the robot footprint leaving the driveable region
(user decision), so the contact channel goes:
- warehouse_v2.world.sdf: the 47 static contact sensors and the contact plugin are
  removed; the rest of the file is byte-identical and the 56 collision boxes are
  unchanged. The header now says the SDF is the world (edit it directly).
- warehouse_amr.urdf.xacro: the body contact sensor is removed.
- bringup_sim: the per-sensor contact bridge, contact_evidence_node and the
  bridge_contacts argument are removed; launch helpers no longer pass it.
- campaign_runner: no contact/geometric collision completion reason.
- Both templates use warehouse_v2.world.sdf; the fast world (which only lowered the
  contact rate) and the shipout world lose their profiles and task alias.
- World contract test: single world, no contact sensors, and every occluder box lies
  inside a declared zone of world/warehouse_v2.py (1 mm tolerance: the SDF writes
  millimetres), the only other boxes being the profile's five included objects.

The experiment logger's contact channel is removed in the next commit.

Co-Authored-By: Claude Opus 5.5 <noreply@anthropic.com>

File: src/sim/robot_description/urdf/warehouse_amr.urdf.xacro (robot description, xacro)
@@ -238,17 +238,4 @@
     </gazebo>
   </xacro:if>
-  <!-- Robot-side physical evidence covers contacts with collision-bearing
-       included props as well as world links. The body collision is the outer
-       obstacle-striking hull; wheel/caster sensors would continuously report
-       normal ground support and obscure obstacle events. -->
-  <gazebo reference="${ns}base_link">
-    <sensor name="body_contact" type="contact">
-      <!-- sdformat lumps the fixed base_joint into base_footprint and assigns
-           this deterministic collision name (verified with `ign sdf -p`). -->
-      <contact><collision>${ns}base_footprint_fixed_joint_lump__base_link_collision</collision></contact>
-      <update_rate>10</update_rate>
-      <always_on>true</always_on>
-    </sensor>
-  </gazebo>
   <!-- ================= Gazebo Harmonic DiffDrive ================= -->
   <gazebo>
